Commit message: fix tf trans which gives me better final goal visualized&make run_pipeline bash

File: src/tools/kinect_description/urdf/kinect/kinect.xacro (robot description, xacro)
@@ -3,5 +3,5 @@
     <xacro:macro name="sensor_kinect" params="prefix name parent cam_px cam_py cam_pz cam_or cam_op cam_oy">
         <!-- Kinect sensor URDF part, cf. https://github.com/turtlebot/turtlebot
-        and there turtlebot_description/urdf/sensors/kinect.xacro -->
+    and there turtlebot_description/urdf/sensors/kinect.xacro -->
         <joint name="${name}_rgb_joint" type="fixed">
             <parent link="${parent}"/>
@@ -13,5 +13,6 @@
             <parent link="${name}_rgb_frame"/>
             <child link="${name}_rgb_optical_frame"/>
-            <origin xyz="0 0 0" rpy="0 0 0"/>
+            <!-- Rotate into REP103 optical frame: roll=-90deg, yaw=-90deg -->
+            <origin xyz="0 0 0" rpy="-1.57 0 -1.57"/>
         </joint>
         <link name="${name}_rgb_optical_frame"/>
